Commit message: 65b compatible with both grippers

File: ros2_rm_robot/dual_rm_description/dual_rm_description/urdf/arms/65b/joints.urdf.xacro (robot description, xacro)
@@ -43,39 +43,42 @@
       xyz="0 0 0" />
   </joint>
-  <joint
-    name="r_hand_joint"
-    type="fixed">
-    <origin
-      xyz="0 0 0.0445"
-      rpy="0 0 0" />
-    <parent
-      link="r_link6" />
-    <child
-      link="r_hand_base_link" />
-    <axis
-      xyz="0 0 -1" />
-    <limit
-      lower="0"
-      upper="0"
-      effort="0"
-      velocity="0" />
-  </joint>
-  <joint
-    name="l_hand_joint"
-    type="fixed">
-    <origin
-      xyz="0 0 0.0445"
-      rpy="3.1415 3.1415 3.1415" />
-    <parent
-      link="l_link6" />
-    <child
-      link="l_hand_base_link" />
-    <axis
-      xyz="0 0 0" />
-    <limit
-      lower="0"
-      upper="0"
-      effort="0"
-      velocity="0" />
-  </joint>
+  <!-- Dummy Hand Joints Wrapped in Conditional -->
+  <xacro:if value="${'$(arg gripper_type)' == 'dummy'}">
+    <joint
+      name="r_hand_joint"
+      type="fixed">
+      <origin
+        xyz="0 0 0.0445"
+        rpy="0 0 0" />
+      <parent
+        link="r_link6" />
+      <child
+        link="r_hand_base_link" />
+      <axis
+        xyz="0 0 -1" />
+      <limit
+        lower="0"
+        upper="0"
+        effort="0"
+        velocity="0" />
+    </joint>
+    <joint
+      name="l_hand_joint"
+      type="fixed">
+      <origin
+        xyz="0 0 0.0445"
+        rpy="3.1415 3.1415 3.1415" />
+      <parent
+        link="l_link6" />
+      <child
+        link="l_hand_base_link" />
+      <axis
+        xyz="0 0 0" />
+      <limit
+        lower="0"
+        upper="0"
+        effort="0"
+        velocity="0" />
+    </joint>
+  </xacro:if>
 </robot>

File: ros2_rm_robot/dual_rm_description/dual_rm_description/urdf/r2d3_description.urdf.xacro (robot description, xacro)
@@ -3,4 +3,6 @@
     <xacro:arg name="arm_model" default="65b"/>
     <xacro:property name="arm_model" value="$(arg arm_model)"/>
+    <xacro:arg name="gripper_type" default="$(optenv GRIPPER_TYPE dummy)"/>
+    <xacro:property name="gripper_type" value="$(arg gripper_type)"/>
     <!-- ═══════════════════════════════════════════════════════════
          Shared components (identical for both arm variants)
@@ -14,8 +16,28 @@
          ═══════════════════════════════════════════════════════════ -->
     <xacro:include filename="$(find dual_rm_description)/urdf/arms/$(arg arm_model)/left_arm.urdf.xacro"/>
-    <xacro:include filename="$(find dual_rm_description)/urdf/arms/$(arg arm_model)/left_hand.urdf.xacro"/>
     <xacro:include filename="$(find dual_rm_description)/urdf/arms/$(arg arm_model)/right_arm.urdf.xacro"/>
-    <xacro:include filename="$(find dual_rm_description)/urdf/arms/$(arg arm_model)/right_hand.urdf.xacro"/>
     <xacro:include filename="$(find dual_rm_description)/urdf/arms/$(arg arm_model)/joints.urdf.xacro"/>
+    <!-- ═══════════════════════════════════════════════════════════
+         Gripper Selection (selected by gripper_type argument)
+         ═══════════════════════════════════════════════════════════ -->
+    <xacro:if value="${gripper_type == 'dummy'}">
+        <!-- Load the original dummy hands -->
+        <xacro:include filename="$(find dual_rm_description)/urdf/arms/$(arg arm_model)/left_hand.urdf.xacro"/>
+        <xacro:include filename="$(find dual_rm_description)/urdf/arms/$(arg arm_model)/right_hand.urdf.xacro"/>
+    </xacro:if>
+    <xacro:if value="${gripper_type == '4c2'}">
+        <!-- Load the new 4c2 Gripper Macro -->
+        <xacro:include filename="$(find dual_rm_description)/urdf/grippers/4c2_gripper.urdf.xacro"/>
+        <!-- Attach to the 6th link for the 65b model -->
+        <xacro:if value="${arm_model == '65b'}">
+            <xacro:gripper_4c2 prefix="l_" parent_link="l_link6" />
+            <xacro:gripper_4c2 prefix="r_" parent_link="r_link6" />
+        </xacro:if>
+        <!-- Attach to the 7th link for the 75b model -->
+        <xacro:if value="${arm_model == '75b'}">
+            <xacro:gripper_4c2 prefix="l_" parent_link="l_link7" />
+            <xacro:gripper_4c2 prefix="r_" parent_link="r_link7" />
+        </xacro:if>
+    </xacro:if>
     <!-- ═══════════════════════════════════════════════════════════
          Transmissions (Only Useful For Gazebo Classic)
