Commit message: 75b compatible with both grippers

File: ros2_rm_robot/dual_rm_description/dual_rm_description/urdf/arms/75b/joints.urdf.xacro (robot description, xacro)
@@ -1,5 +1,5 @@
 <?xml version="1.0"?>
 <robot name="joint" xmlns:xacro="http://www.ros.org/wiki/xacro">
-   <joint
+  <joint
     name="body_base_joint"
     type="fixed">
@@ -43,39 +43,42 @@
       xyz="0 0 0" />
   </joint>
-  <joint
-    name="r_hand_joint"
-    type="fixed">
-    <origin
-      xyz="0 0 0.0445"
-      rpy="0 0 0" />
-    <parent
-      link="r_link7" />
-    <child
-      link="r_hand" />
-    <axis
-      xyz="0 0 -1" />
-    <limit
-      lower="0"
-      upper="0"
-      effort="0"
-      velocity="0" />
-  </joint>
-  <joint
-    name="l_hand_joint"
-    type="fixed">
-    <origin
-      xyz="0 0 0.0445"
-      rpy="0 0 3.1415" />
-    <parent
-      link="l_link7" />
-    <child
-      link="l_hand_link" />
-    <axis
-      xyz="0 0 0" />
-    <limit
-      lower="0"
-      upper="0"
-      effort="0"
-      velocity="0" />
-  </joint>
+  <!-- Dummy Hand Joints Wrapped in Conditional -->
+  <xacro:if value="${'$(arg gripper_type)' == 'dummy'}">
+    <joint
+      name="r_hand_joint"
+      type="fixed">
+      <origin
+        xyz="0 0 0.0445"
+        rpy="0 0 0" />
+      <parent
+        link="r_link7" />
+      <child
+        link="r_hand" />
+      <axis
+        xyz="0 0 -1" />
+      <limit
+        lower="0"
+        upper="0"
+        effort="0"
+        velocity="0" />
+    </joint>
+    <joint
+      name="l_hand_joint"
+      type="fixed">
+      <origin
+        xyz="0 0 0.0445"
+        rpy="0 0 3.1415" />
+      <parent
+        link="l_link7" />
+      <child
+        link="l_hand_link" />
+      <axis
+        xyz="0 0 0" />
+      <limit
+        lower="0"
+        upper="0"
+        effort="0"
+        velocity="0" />
+    </joint>
+  </xacro:if>
 </robot>
