Commit message: mujoco sim working with all configurations of arms and grippers

File: ros2_rm_robot/dual_rm_description/dual_rm_description/urdf/grippers/4c2_gripper.urdf.xacro (robot description, xacro)
@@ -324,64 +324,70 @@
     <material>Gazebo/Grey</material>
   </gazebo>
-  <!-- Only load the Gazebo control plugin if use_gazebo is true -->
-  <xacro:if value="$(arg use_gazebo)">
-    <ros2_control name="${prefix}Gripper_Hardware" type="system">
-      <hardware>
+  <!-- ═══════════════════════════════════════════════════════════
+       ROS 2 Control (Hardware Interfaces)
+       ═══════════════════════════════════════════════════════════ -->
+  <ros2_control name="${prefix}Gripper_Hardware" type="system">
+    <hardware>
+      <xacro:if value="$(arg use_gazebo)">
         <plugin>gz_ros2_control/GazeboSimSystem</plugin>
-      </hardware>
-      <joint name="${prefix}gripper_joint">
-        <param name="pos_kp">5.0</param>
-        <param name="pos_ki">0.0</param>
-        <param name="pos_kd">0.1</param>
-        <param name="pos_max_integral_error">1.0</param>
-        <command_interface name="position"/>
-        <state_interface name="position">
-          <param name="initial_value">0.0</param>
-        </state_interface>
-        <state_interface name="velocity"/>
-        <state_interface name="effort"/>
-      </joint>
-      <joint name="${prefix}r_3_joint">
-        <command_interface name="position">
-          <param name="min">0</param>
-          <param name="max">1.0</param>
-        </command_interface>
-        <state_interface name="position"/>
-        <state_interface name="velocity"/>
-      </joint>
-      <joint name="${prefix}l_1_joint">
-        <command_interface name="position">
-          <param name="min">0</param>
-          <param name="max">1.0</param>
-        </command_interface>
-        <state_interface name="position"/>
-        <state_interface name="velocity"/>
-      </joint>
-      <joint name="${prefix}l_3_joint">
-        <command_interface name="position">
-          <param name="min">0</param>
-          <param name="max">1.0</param>
-        </command_interface>
-        <state_interface name="position"/>
-        <state_interface name="velocity"/>
-      </joint>
-      <joint name="${prefix}r_2_joint">
-        <command_interface name="position">
-          <param name="min">0</param>
-          <param name="max">1.0</param>
-        </command_interface>
-        <state_interface name="position"/>
-        <state_interface name="velocity"/>
-      </joint>
-      <joint name="${prefix}l_2_joint">
-        <command_interface name="position">
-          <param name="min">0</param>
-          <param name="max">1.0</param>
-        </command_interface>
-        <state_interface name="position"/>
-        <state_interface name="velocity"/>
-      </joint>
-    </ros2_control>
-  </xacro:if>
+      </xacro:if>
+      <xacro:unless value="$(arg use_gazebo)">
+        <!-- Use a mock system to prevent MuJoCo from spawning multiple physics instances -->
+        <plugin>mock_components/GenericSystem</plugin>
+      </xacro:unless>
+    </hardware>
+    <joint name="${prefix}gripper_joint">
+      <param name="pos_kp">5.0</param>
+      <param name="pos_ki">0.0</param>
+      <param name="pos_kd">0.1</param>
+      <param name="pos_max_integral_error">1.0</param>
+      <command_interface name="position"/>
+      <state_interface name="position">
+        <param name="initial_value">0.0</param>
+      </state_interface>
+      <state_interface name="velocity"/>
+      <state_interface name="effort"/>
+    </joint>
+    <joint name="${prefix}r_3_joint">
+      <command_interface name="position">
+        <param name="min">0</param>
+        <param name="max">1.0</param>
+      </command_interface>
+      <state_interface name="position"/>
+      <state_interface name="velocity"/>
+    </joint>
+    <joint name="${prefix}l_1_joint">
+      <command_interface name="position">
+        <param name="min">0</param>
+        <param name="max">1.0</param>
+      </command_interface>
+      <state_interface name="position"/>
+      <state_interface name="velocity"/>
+    </joint>
+    <joint name="${prefix}l_3_joint">
+      <command_interface name="position">
+        <param name="min">0</param>
+        <param name="max">1.0</param>
+      </command_interface>
+      <state_interface name="position"/>
+      <state_interface name="velocity"/>
+    </joint>
+    <joint name="${prefix}r_2_joint">
+      <command_interface name="position">
+        <param name="min">0</param>
+        <param name="max">1.0</param>
+      </command_interface>
+      <state_interface name="position"/>
+      <state_interface name="velocity"/>
+    </joint>
+    <joint name="${prefix}l_2_joint">
+      <command_interface name="position">
+        <param name="min">0</param>
+        <param name="max">1.0</param>
+      </command_interface>
+      <state_interface name="position"/>
+      <state_interface name="velocity"/>
+    </joint>
+  </ros2_control>
   </xacro:macro>
 </robot>
